File: Hardware Design/PCBs/MITCH_2021-48/PSPS_AVNC_SRD_CS_combined-2021-02-07.brd (EAGLE design)
At the start: 129.8 x 132.6 mm, 15 parts, among them U0-C STM32F411CEUX, U0-S TPS62202

Commit message: further nand debugging
Routing:
- net SPI2R_SCK: track 6.79 -> 9.43 mm
Changed lines of the file:
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@@
 <drawing>
 <settings>
-<setting alwaysvectorfont="yes"/>
+<setting alwaysvectorfont="no"/>
 <setting verticaltext="up"/>
 </settings>
@@
 <wire x1="12.25" y1="-0.75" x2="13.75" y2="-0.75" width="0.127" layer="2"/>
 <wire x1="15.4999" y1="0.9999" x2="13.75" y2="-0.75" width="0.127" layer="2"/>
+<wire x1="15.4999" y1="2.54" x2="14.5399" y2="3.5" width="0.1524" layer="2"/>
+<wire x1="14.5399" y1="3.5" x2="13.25" y2="3.5" width="0.1524" layer="2"/>
 </signal>
 <signal name="SPI2R_MOSI">
